File: psu/psu.kicad_sch (KiCad schematic)
At the start: 0 parts

Commit message: semi finished the schematic , next up anotation and PCB layout
Parts:
- added C1, C2, C4, C5: 4.7u, symbol Device:C_Small
- added C3: 1u, symbol Device:C_Small
- added D1: LED_Small, symbol Device:LED_Small
- added J1, J2: Screw_Terminal_01x02, symbol Connector:Screw_Terminal_01x02
- added NT1: NetTie_2, symbol Device:NetTie_2
- added R1: 10K, symbol Device:R_Small
- added R2: 22K, symbol Device:R_Small
- added R3: R_Small, symbol Device:R_Small
- added R4, R5: (no value), symbol Device:R_Small
- added U1: (no value), halfgeleiders:TLVM13630, symbol Halfgelijders:TLVM13630
Connections:
- new net: C3.2, R4.1, R5.1, U1.26 (PG)
- new net: C3.1, R4.2, U1.23 (VCC)
- new net: C1.1, C2.1, J1.2 (Pin_2), U1.18 (VIN), U1.19 (VIN), U1.2 (EN), U1.3 (VIN), U1.4 (VIN)
- new net: R2.2, U1.1 (RT)
- new net: C4.1, C5.1, J2.1 (Pin_1), R3.1, U1.10 (VOUT), U1.12 (VOUT), U1.13 (VOUT), U1.14 (VOUT), U1.15 (VOUT), U1.7 (VOUT), U1.8 (VOUT), U1.9 (VOUT)
- new net: R1.1, R3.2, U1.25 (FB)
- new net: D1.2 (A), R5.2
- new net AGND: NT1.1, R1.2, R2.1, U1.24 (AGND)
- new net PGND: C1.2, C2.2, C4.2, C5.2, D1.1 (K), J1.1 (Pin_1), J2.2 (Pin_2), NT1.2, U1.16 (PGND), U1.17 (PGND), U1.5 (PGND), U1.6 (PGND)
- no-connect marks 0 -> 2
Other:
- added sheet documentation (documentation.kicad_sch)
- note added: "Calculation for the upper resistor, Rfb is recomended at 10K"
- note added: "RT"

Commit message: added bom and finished the schematic , board will be a pita
Parts:
- added R6: (no value), Resistor_SMD:R_0201_0603Metric_Pad0.64x0.40mm_HandSolder, symbol Device:R_Small
- added R7: 0, Resistor_SMD:R_0201_0603Metric_Pad0.64x0.40mm_HandSolder, symbol Device:R_Small
- C1, C2, C4, C5: footprint (none) -> vanalles:0603; Digikey MPN (none) -> 87-MSASJ168BB7475MTNA01CT-ND; Digikey price/pcs (none) -> 0,31 €; LCSC MPN (none) -> C22399629; LCSC price/pcs (none) -> 0.27 €; Mouser MPN (none) -> 963-MLASJ168BB7475KT; Mouser price/pcs (none) -> 0,32 €
- C3: footprint (none) -> Capacitor_SMD:C_0201_0603Metric; Digikey MPN (none) -> 587-MCAST063SB7222KFCA1JTR-ND; Digikey price/pcs (none) -> 0,01125 €; LCSC MPN (none) -> /; LCSC price/pcs (none) -> 0 €; Mouser MPN (none) -> 963-E063SB7222KFCA1J; Mouser price/pcs (none) -> 0,10 €
- D1: footprint (none) -> LED_SMD:LED_0201_0603Metric
- J1: footprint (none) -> TerminalBlock:TerminalBlock_Xinya_XY308-2.54-2P_1x02_P2.54mm_Horizontal; now left out of the parts list
- J2: footprint (none) -> TerminalBlock:TerminalBlock_Xinya_XY308-2.54-2P_1x02_P2.54mm_Horizontal
- NT1: footprint (none) -> NetTie:NetTie-2_SMD_Pad0.5mm
- R1: footprint (none) -> Resistor_SMD:R_0201_0603Metric_Pad0.64x0.40mm_HandSolder; Digikey MPN (none) -> P10KBXCT-ND; Digikey price/pcs (none) -> 0,10 €; LCSC MPN (none) -> C490808; LCSC price/pcs (none) -> 0.124 €; Mouser MPN (none) -> 667-ERA-1AEB103C; Mouser price/pcs (none) -> 0,10 €
- R2: footprint (none) -> Resistor_SMD:R_0201_0603Metric_Pad0.64x0.40mm_HandSolder; Digikey MPN (none) -> 408-RG0603P-223-D-T10CT-ND; Digikey price/pcs (none) -> 0,15 €; LCSC MPN (none) -> C20135502; LCSC price/pcs (none) -> 0,16 €; Mouser MPN (none) -> 754-RG0603P-223-D; Mouser price/pcs (none) -> 0,15 €
- R3: value R_Small -> 34K; footprint (none) -> Resistor_SMD:R_0201_0603Metric_Pad0.64x0.40mm_HandSolder; Digikey MPN (none) -> YAG2614CT-ND; Digikey price/pcs (none) -> 0,09 €; LCSC MPN (none) -> C273307; LCSC price/pcs (none) -> € 0.0009; Mouser MPN (none) -> 603-RC0201FR-0734KL; Mouser price/pcs (none) -> 0,09 €
- R4, R5: footprint (none) -> Resistor_SMD:R_0201_0603Metric_Pad0.64x0.40mm_HandSolder
- U1: Digikey MPN (none) -> 296-TLVM13630RDHRCT-ND; Digikey price/pcs (none) -> 3,36 €; LCSC MPN (none) -> C5219304; LCSC price/pcs (none) -> 4.91 €; Mouser MPN (none) -> 595-TLVM13630RDHR; Mouser price/pcs (none) -> 3,58 €
Connections:
- net AGND: now also R6.2
- net PGND: now also C3.2
- net at R4.1, R5.1, U1.26 (PG): no longer C3.2
- net at C1.1, C2.1, J1.2 (Pin_2)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: now also R7.2; no longer U1.2 (EN)
- new net: R6.1, R7.1, U1.2 (EN)
Other:
- note added: "<Calculated value is 35K, availble value is 34K, calculated Vout is 3.4001"
- note added: "Place capacitors close to the package and must be X7R dielectric or better"
- note added: "RT tabel based on switching frequency based on desired output"
- moved on the sheet: C1, C3, D1, R2, R4, R5

Commit message: made the pcb , It's a bit trash but still need to make a q&a document
Parts:
- C1, C2: footprint vanalles:0603 -> Capacitor_SMD:C_0805_2012Metric; Digikey MPN 87-MSASJ168BB7475MTNA01CT-ND -> 478-KGM21AR71E475KUCT-ND; Digikey price/pcs 0,31 € -> (none); LCSC MPN C22399629 -> C513766; LCSC price/pcs 0.27 € -> 0.0137 €; Mouser MPN 963-MLASJ168BB7475KT -> 581-KGM21AR71E475KU; Mouser price/pcs 0,32 € -> 0,59 €
- D1, J2, R4, R5: now left out of the parts list
Connections:
- net PG: now reaches R4.1, R5.1, U1.26 (PG)
- net VCC: now reaches C3.1, R4.2, U1.23 (VCC)
- net Vin: now reaches C1.1, C2.1, J1.2 (Pin_2), R7.2, U1.18 (VIN), U1.19 (VIN), U1.3 (VIN), U1.4 (VIN)
- net RT: now reaches R2.2, U1.1 (RT)
- net Vout: now reaches C4.1, C5.1, J2.1 (Pin_1), R3.1, U1.10 (VOUT), U1.12 (VOUT), U1.13 (VOUT), U1.14 (VOUT), U1.15 (VOUT), U1.7 (VOUT), U1.8 (VOUT), U1.9 (VOUT)
- net FB: now reaches R1.1, R3.2, U1.25 (FB)
- net EN: now reaches R6.1, R7.1, U1.2 (EN)
Other:
- removed sheet documentation
